File: CAD/Nivelador Láser.kicad_sch (KiCad schematic)
At the start: 7 parts

Commit message: Add files via upload
Parts:
- removed R1: 10k, Resistor_SMD:R_0805_2012Metric_Pad1.20x1.40mm_HandSolder, symbol Device:R
- added Driver1: Motor_Driver, Connector_Wire:SolderWire-0.5sqmm_1x04_P4.6mm_D0.9mm_OD2.1mm_Relief, symbol Connector:Conn_01x04_Male
- added R2: 10k, Resistor_SMD:R_0805_2012Metric_Pad1.20x1.40mm_HandSolder, symbol Device:R
Connections:
- net +5V: now also Driver1.1 (Pin_1), R2.2
- net GND: now also Driver1.2 (Pin_2)
- net HALL: now also UNO1.23 (D8), R2.1
- net IMU_SCL: now also UNO1.14 (SCL/A5); no longer UNO1.13 (SDA/A4)
- net IMU_SDA: now also UNO1.13 (SDA/A4); no longer UNO1.14 (SCL/A5)
- net SV1: now also UNO1.20 (D5)
- net SV2: now also UNO1.21 (D6)
- net LSR: now reaches Laser1.1 (Pin_1)
- net LSR: now also UNO1.22 (D7)
- net MTR: now reaches UNO1.25 (D10)
- net MTR: now also Driver1.3 (Pin_3)
- no-connect marks 4 -> 5
