File: CAD/Receptor Laser/Receptor Laser.kicad_sch (KiCad schematic)
At the start: 115 parts

Commit message: a
Parts:
- removed OP_AMP1, OP_AMP10, OP_AMP11, OP_AMP12, OP_AMP2, OP_AMP3, OP_AMP4, OP_AMP5, OP_AMP6, OP_AMP7, OP_AMP8, OP_AMP9: MC33079, Package_SO:SOIC-14_3.9x8.7mm_P1.27mm, symbol Amplifier_Operational:MC33079
- removed R1, R10, R11, R12, R13, R14, R15, R16, R17, R18, R19, R2, R20, R21, R22, R23, R24, R25, R26, R27, R28, R29, R3, R30, R31, R32, R33, R34, R35, R36, R37, R38, R39, R4, R40, R41, R42, R43, R44, R45, R46, R47, R48, R5, R6, R7, R8, R9: R, Resistor_SMD:R_0805_2012Metric_Pad1.20x1.40mm_HandSolder, symbol Device:R
Connections:
- net PH-1: now also PH1.A
- net PH-10: now also PH10.A
- net PH-11: now also PH11.A
- net PH-12: now also PH12.A
- net PH-13: now also PH13.A
- net PH-14: now also PH14.A
- net PH-15: now also PH15.A
- net PH-16: now also PH16.A
- net PH-17: now also PH17.A
- net PH-18: now also PH18.A
- net PH-19: now also PH19.A
- net PH-2: now also PH2.A
- net PH-20: now also PH20.A
- net PH-21: now also PH21.A
- net PH-22: now also PH22.A
- net PH-23: now also PH23.A
- net PH-24: now also PH24.A
- net PH-25: now also PH25.A
- net PH-26: now also PH26.A
- net PH-27: now also PH27.A
- net PH-28: now also PH28.A
- net PH-29: now also PH29.A
- net PH-3: now also PH3.A
- net PH-30: now also PH30.A
- net PH-31: now also PH31.A
- net PH-32: now also PH32.A
- net PH-33: now also PH33.A
- net PH-34: now also PH34.A
- net PH-35: now also PH35.A
- net PH-36: now also PH36.A
- net PH-37: now also PH37.A
- net PH-38: now also PH38.A
- net PH-39: now also PH39.A
- net PH-4: now also PH4.A
- net PH-40: now also PH40.A
- net PH-41: now also PH41.A
- net PH-42: now also PH42.A
- net PH-43: now also PH43.A
- net PH-44: now also PH44.A
- net PH-45: now also PH45.A
- net PH-46: now also PH46.A
- net PH-47: now also PH47.A
- net PH-48: now also PH48.A
- net PH-5: now also PH5.A
- net PH-6: now also PH6.A
- net PH-7: now also PH7.A
- net PH-8: now also PH8.A
- net PH-9: now also PH9.A
- no-connect marks 0 -> 18
Other:
- moved on the sheet: A1, ADC1, PH1, PH2, PH3, PH4, PH5, PH6, PH7, PH8

Commit message: pcb receptor
Parts:
- renumbered A1 to UNO1
Changed lines of the file:
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@@
 		(dnp no)
 		(fields_autoplaced yes)
-		(property "Reference" "A1"
+		(property "Reference" "UNO1"
 			(at 318.4241 148.59 0)
 			(effects
@@
 			(project ""
 				(path "/a079cfad-514e-45ca-915a-9427d80cf52d"
-					(reference "A1")
+					(reference "UNO1")
 					(unit 1)
 				)
