File: CAD/Receptor Laser/Receptor Laser.kicad_sch (KiCad schematic)
At the start: 57 parts

Commit message: a
Parts:
- BZ1: footprint Buzzer_Beeper:Buzzer_TDK_PS1240P02BT_D12.2mm_H6.5mm -> Buzzer_Beeper:Buzzer_12x9.5RM7.6
Connections:
- net BUZZ: now also UNO1.18 (D3)
- no-connect marks 16 -> 15
Changed lines of the file:
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@@
 	)
 	(no_connect
-		(at 298.45 168.91)
-	)
-	(no_connect
 		(at 298.45 171.45)
 	)
@@
 	(wire
 		(pts
+			(xy 292.1 168.91) (xy 298.45 168.91)
+		)
+		(stroke
+			(width 0)
+			(type default)
+		)
+	)
+	(wire
+		(pts
 			(xy 77.47 233.68) (xy 77.47 234.95)
 		)
@@
 		)
 	)
+	(label "BUZZ"
+		(at 292.1 168.91 0)
+		(fields_autoplaced yes)
+		(effects
+			(font
+				(size 1.27 1.27)
+			)
+			(justify left bottom)
+		)
+	)
 	(label "PH-41"
 		(at 205.74 275.59 0)
@@
 			)
 		)
-		(property "Footprint" "Buzzer_Beeper:Buzzer_TDK_PS1240P02BT_D12.2mm_H6.5mm"
+		(property "Footprint" "Buzzer_Beeper:Buzzer_12x9.5RM7.6"
 			(at 306.705 247.65 90)
 			(effects
