File: CAD/Nivelador Laser/Nivelador Laser.kicad_sch (KiCad schematic)
At the start: 8 parts

Commit message: changes
Connections:
- no-connect marks 5 -> 25
Changed lines of the file:
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@@
+	)
+	(no_connect
+		(at 158.75 110.49)
 	)
 	(no_connect
@@
 	)
 	(no_connect
+		(at 168.91 72.39)
+	)
+	(no_connect
 		(at 63.5 149.86)
+	)
+	(no_connect
+		(at 184.15 100.33)
+	)
+	(no_connect
+		(at 158.75 92.71)
+	)
+	(no_connect
+		(at 184.15 87.63)
+	)
+	(no_connect
+		(at 184.15 115.57)
+	)
+	(no_connect
+		(at 158.75 113.03)
+	)
+	(no_connect
+		(at 158.75 85.09)
+	)
+	(no_connect
+		(at 184.15 118.11)
+	)
+	(no_connect
+		(at 158.75 82.55)
+	)
+	(no_connect
+		(at 184.15 102.87)
+	)
+	(no_connect
+		(at 158.75 107.95)
+	)
+	(no_connect
+		(at 184.15 92.71)
+	)
+	(no_connect
+		(at 158.75 115.57)
+	)
+	(no_connect
+		(at 184.15 97.79)
 	)
 	(no_connect
@@
 	)
 	(no_connect
+		(at 184.15 105.41)
+	)
+	(no_connect
+		(at 158.75 87.63)
+	)
+	(no_connect
+		(at 184.15 82.55)
+	)
+	(no_connect
 		(at 63.5 152.4)
 	)
+	(no_connect
+		(at 158.75 90.17)
+	)
+	(no_connect
+		(at 173.99 72.39)
+	)
 	(wire

Commit message: a
Parts:
- removed Driver1: Motor_Driver, Connector_Wire:SolderWire-0.5sqmm_1x04_P4.6mm_D0.9mm_OD2.1mm_Relief, symbol Connector:Conn_01x04_Pin
- removed Hall1: Hall_Sensor, Connector_Wire:SolderWire-0.5sqmm_1x03_P4.6mm_D0.9mm_OD2.1mm_Relief, symbol Connector:Conn_01x03_Pin
- removed IMU1: MPU-6050, Connector_PinSocket_2.54mm:PinSocket_1x08_P2.54mm_Vertical, symbol Connector:Conn_01x08_Pin
- removed R1: 10k, Resistor_SMD:R_0805_2012Metric_Pad1.20x1.40mm_HandSolder, symbol Device:R
- added BT1: ZS-040, symbol Connector:Conn_01x05_Male
- added IMU1: MPU-6050, Connector_PinSocket_2.54mm:PinSocket_1x04_P2.54mm_Vertical, symbol Connector:Conn_01x04_Male
Connections:
- net +5V: now also BT1.3 (Pin_3), IMU1.1 (Pin_1)
- net GND: now also BT1.4 (Pin_4), IMU1.2 (Pin_2)
- net IMU_SCL: now also IMU1.3 (Pin_3)
- net IMU_SDA: now also IMU1.4 (Pin_4)
- net HALL renamed BT_RX
- net BT_RX: now also BT1.1 (Pin_1)
- net MTR renamed BT_TX
- net BT_TX: now also BT1.2 (Pin_2)
- no-connect marks 25 -> 21

Commit message: a
Parts:
- removed BT1: ZS-040, symbol Connector:Conn_01x05_Male
Connections:
- net BT_RX: no longer names the net of UNO1.23 (D8)
- net BT_TX: no longer names the net of UNO1.24 (D9)
- no-connect marks 21 -> 22
